File: ethernet.kicad_sch (KiCad schematic)
At the start: 6 parts, among them J6 5-2337992-8

Commit message: Renaming Sheets
Other:
- company: Antmicro Ltd -> Dronolab
- title: Jetson Orin Baseboard -> Ethernet
Changed lines of the file:
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@@
   (paper "A3")
   (title_block
-    (title "Jetson Orin Baseboard")
-    (date "2023-03-03")
-    (rev "1.1.0")
-    (company "Antmicro Ltd")
-    (comment 1 "www.antmicro.com")
+    (title "Ethernet")
+    (date "2023-07-05")
+    (rev "1.0.0")
+    (company "Dronolab")
+    (comment 1 "dronolab.etsmtl.ca")
   )
   (junction (at 182.88 166.37) (diameter 0) (color 0 0 0 0)
