File: m-2.kicad_sch (KiCad schematic)
At the start: 61 parts, among them J1 2199230-6, J2 1-2199230-6, M2 M2_4222, M3 M2_2280, U2 74LVC2G07GV, U3 74LVC2G07GV, Y1 ECS-327MVATX-2-CN-TR3

Commit message: Renaming Sheets
Other:
- company: Antmicro Ltd -> Dronolab
- title: Jetson Orin Baseboard -> M.2
Changed lines of the file:
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@@
   (paper "A3")
   (title_block
-    (title "Jetson Orin Baseboard")
-    (date "2023-03-03")
-    (rev "1.1.0")
-    (company "Antmicro Ltd")
-    (comment 1 "www.antmicro.com")
+    (title "M.2")
+    (date "2023-07-05")
+    (rev "1.0.0")
+    (company "Dronolab")
+    (comment 1 "dronolab.etsmtl.ca")
   )
   (junction (at 345.44 115.57) (diameter 0) (color 0 0 0 0)
