File: hdmi.kicad_sch (KiCad schematic)
At the start: 58 parts, among them J13 WE_685119136923_alt_sym, Q1 PJE138K, Q12 PJE138K, Q2 PJE138K, Q3 PJE138K, U36 TS3DV642RUARQ1, U43 NTS0102GT, U44 TPD4E05U06QDQARQ1, U45 TPD4E05U06QDQARQ1, U46 TPD4E05U06QDQARQ1

Commit message: Renaming Sheets
Other:
- company: Antmicro Ltd -> Dronolab
- title: Jetson Orin Baseboard -> HDMI
Changed lines of the file:
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@@
   (paper "A3")
   (title_block
-    (title "Jetson Orin Baseboard")
-    (date "2023-03-03")
-    (rev "1.1.0")
-    (company "Antmicro Ltd")
-    (comment 1 "www.antmicro.com")
+    (title "HDMI")
+    (date "2023-07-05")
+    (rev "1.0.0")
+    (company "Dronolab")
+    (comment 1 "dronolab.etsmtl.ca")
   )
   (junction (at 378.46 187.96) (diameter 0) (color 0 0 0 0)
