File: csi.kicad_sch (KiCad schematic)
At the start: 65 parts, among them J7 WE_68715014522_ONE-SIDE, J8 WE_68715014522_ONE-SIDE, U24 AP22615, U25 AP22615, U26 PI4MSD5V9548AZDEX, U27 AP22615, U28 AP22615, U31 NTS0102GT, U32 NTS0102GT

Commit message: Renaming Sheets
Other:
- company: Antmicro Ltd -> Dronolab
- title: Jetson Orin Baseboard -> CSI
Changed lines of the file:
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@@
   (paper "A3")
   (title_block
-    (title "Jetson Orin Baseboard")
-    (date "2023-03-03")
-    (rev "1.1.0")
-    (company "Antmicro Ltd")
-    (comment 1 "www.antmicro.com")
+    (title "CSI")
+    (date "2023-07-05")
+    (rev "1.0.0")
+    (company "Dronolab")
+    (comment 1 "dronolab.etsmtl.ca")
   )
   (junction (at 360.68 96.52) (diameter 0) (color 0 0 0 0)

Commit message: Changes to CSI for multiplexing and to peripherals for better PAC connector
Parts:
- removed C94, C95, C98, C99: C_1u_0402, jetson-orin-baseboard-footprints:0402-cap, symbol jetson-orin-baseboard:C_1u_0402
- removed D18, D20, D24, D25: LTST-C190GKT, jetson-orin-baseboard-footprints:LED_0603, symbol jetson-orin-baseboard:LTST-C190GKT
- removed J7, J8: WE_68715014522_ONE-SIDE, jetson-orin-baseboard-footprints:WE_68715014522_ONE-SIDE, symbol jetson-orin-baseboard:WE_68715014522_ONE-SIDE
- removed R103, R107, R108, R122, R50, R51: 4x0R_0201_array, jetson-orin-baseboard-footprints:EXB18V, symbol jetson-orin-baseboard:4x0R_0201_array
- removed R132, R133: R_200R_0402, jetson-orin-baseboard-footprints:0402-res, symbol jetson-orin-baseboard:R_200R_0402
- removed R197, R206: R_470R_0402, jetson-orin-baseboard-footprints:0402-res, symbol jetson-orin-baseboard:R_470R_0402
- removed TP36, TP37, TP38, TP39, TP40, TP41, TP42, TP43: TP_SMD_0_75MM, jetson-orin-baseboard-footprints:Testpoint_smd_0_75mm, symbol jetson-orin-baseboard:TP_SMD_0_75MM
- added C131, C132, C88, C92: C_100n_0402, jetson-orin-baseboard-footprints:0402-cap, symbol jetson-orin-baseboard:C_100n_0402
- added C133, C135: 1u, symbol Device:C
- added R105, R142: R_100k_0402, jetson-orin-baseboard-footprints:0402-res, symbol jetson-orin-baseboard:R_100k_0402
- added R117, R129, R144, R78: R_10k_0402, jetson-orin-baseboard-footprints:0402-res, symbol jetson-orin-baseboard:R_10k_0402
- added R123, R127, R145, R146: R_4k7_0402, jetson-orin-baseboard-footprints:0402-res, symbol jetson-orin-baseboard:R_4k7_0402
- added R148, R149, R50, R51: 10k, symbol Device:R
- added R47, R49, R74, R76: R_0R_0402, jetson-orin-baseboard-footprints:0402-res, symbol jetson-orin-baseboard:R_0R_0402
- added R52, R77: 4x2k2_0201_array, jetson-orin-baseboard-footprints:EXB18V, symbol jetson-orin-baseboard:4x2k2_0201_array
- added U11, U23, U36, U9: AP22615, jetson-orin-baseboard-footprints:TSOT23-6, symbol jetson-orin-baseboard:AP22615
- added U39, U40: TS3DV642RUARQ1, jetson-orin-baseboard-footprints:WQFN-42-1EP_3.5x9mm_P0.5mm_EP2.05x7.55mm, symbol jetson-orin-baseboard:TS3DV642RUARQ1
Connections:
- net +1V8: now also R49.2, R76.2
- net +3V3: now also C132.1, C133.1, C135.1, C92.1, R117.1, R129.2, R144.1, R148.1, R149.1, R47.2, R50.1, R51.1, R74.2, R78.2, U11.6 (IN), U36.6 (IN), U39.1 (VCC), U40.1 (VCC)
- net +5V: now also C131.1, C88.1, U23.6 (IN), U9.6 (IN)
- net CSI0_CLK_N: now also U39.6 (D0-)
- net CSI0_CLK_P: now also U39.5 (D0+)
- net CSI0_D0_N: now also U39.8 (D1-)
- net CSI0_D0_P: now also U39.7 (D1+)
- net CSI0_D1_N: now also U39.11 (D2-)
- net CSI0_D1_P: now also U39.10 (D2+)
- net CSI1_CLK_N: now also U39.13 (D3-)
- net CSI1_CLK_P: now also U39.12 (D3+)
- net CSI1_D0_N: now also U39.4 (SDA/AUX-)
- net CSI1_D0_P: now also U39.3 (SCL/AUX+)
- net CSI1_D1_N: now also U39.15 (CEC)
- net CSI1_D1_P: now also U39.14 (HPD)
- net CSI2_CLK_N: now also U40.6 (D0-)
- net CSI2_CLK_P: now also U40.5 (D0+)
- net CSI2_D0_N: now also U40.8 (D1-)
- net CSI2_D0_P: now also U40.7 (D1+)
- net CSI2_D1_N: now also U40.11 (D2-)
- net CSI2_D1_P: now also U40.10 (D2+)
- net CSI3_CLK_N: now also U40.13 (D3-)
- net CSI3_CLK_P: now also U40.12 (D3+)
- net CSI3_D0_N: now also U40.4 (SDA/AUX-)
- net CSI3_D0_P: now also U40.3 (SCL/AUX+)
- net CSI3_D1_N: now also U40.15 (CEC)
- net CSI3_D1_P: now also U40.14 (HPD)
- net GND: now also C131.2, C132.2, C133.2, C135.2, C88.2, C92.2, R105.1, R123.1, R127.1, R142.1, R145.1, R146.1, U11.2 (GND), U23.2 (GND), U36.2 (GND), U39.43 (GND), U40.43 (GND), U9.2 (GND)
- net MUX_I2C_4_SCL renamed SCL_CAM4
- net SCL_CAM4: now also R52.3
- net MUX_I2C_4_SDA renamed SDA_CAM4
- net SDA_CAM4: now also R52.4
- net MUX_I2C_5_SCL renamed SCL_CAM5
- net SCL_CAM5: now also R52.1
- net MUX_I2C_5_SDA renamed SDA_CAM5
- net SDA_CAM5: now also R52.2
- net MUX_I2C_6_SCL renamed SCL_CAM6
- net SCL_CAM6: now also R77.3
- net MUX_I2C_6_SDA renamed SDA_CAM6
- net SDA_CAM6: now also R77.4
- net MUX_I2C_7_SCL renamed SCL_CAM7
- net SCL_CAM7: now also R77.1
- net MUX_I2C_7_SDA renamed SDA_CAM7
- net SDA_CAM7: now also R77.2
- new net: R51.2, U39.16 (SEL1)
- new net: R50.2, U40.16 (SEL1)
- new net CSIC_3V3: U11.1 (OUT)
- new net CSIC_3V3_ISET: R127.2, U11.5 (ISET)
- new net CSIC_5V: U9.1 (OUT)
- new net CSIC_5V_ISET: R123.2, U9.5 (ISET)
- new net CSIC_FLG: R117.2, U11.3 (FLG), U9.3 (FLG)
- new net CSIC_I2C_VCC: R47.1, R49.1, R52.5, R52.6, R52.7, R52.8
- new net CSIC_PEN: R105.2, R78.1, U11.4 (EN), U9.4 (EN)
- new net CSID_3V3: U36.1 (OUT)
- new net CSID_3V3_ISET: R146.2, U36.5 (ISET)
- new net CSID_5V: U23.1 (OUT)
- new net CSID_5V_ISET: R145.2, U23.5 (ISET)
- new net CSID_FLG: R144.2, U23.3 (FLG), U36.3 (FLG)
- new net CSID_I2C_VCC: R74.1, R76.1, R77.5, R77.6, R77.7, R77.8
- new net CSID_PEN: R129.1, R142.2, U23.4 (EN), U36.4 (EN)
- new net CSI_CAM_0_CLK_N: U39.37 (D0-A)
- new net CSI_CAM_0_CLK_P: U39.38 (D0+A)
- new net CSI_CAM_0_D0_N: U39.35 (D1-A)
- new net CSI_CAM_0_D0_P: U39.36 (D1+A)
- new net CSI_CAM_0_D1_N: U39.33 (D2-A)
- new net CSI_CAM_0_D1_P: U39.34 (D2+A)
- new net CSI_CAM_1_CLK_N: U39.31 (D3-A)
- new net CSI_CAM_1_CLK_P: U39.32 (D3+A)
- new net CSI_CAM_1_D0_N: U39.41 (SDA/AUX-_A)
- new net CSI_CAM_1_D0_P: U39.42 (SCL/AUX+_A)
- new net CSI_CAM_1_D1_N: U39.19 (HPD_A)
- new net CSI_CAM_1_D1_P: U39.18 (CEC_A)
- new net CSI_CAM_2_CLK_N: U39.28 (D0-B)
- new net CSI_CAM_2_CLK_P: U39.29 (D0+B)
- new net CSI_CAM_2_D0_N: U39.26 (D1-B)
- new net CSI_CAM_2_D0_P: U39.27 (D1+B)
- new net CSI_CAM_2_D1_N: U39.24 (D2-B)
- new net CSI_CAM_2_D1_P: U39.25 (D2+B)
- new net CSI_CAM_3_CLK_N: U39.22 (D3-B)
- new net CSI_CAM_3_CLK_P: U39.23 (D3+B)
- new net CSI_CAM_3_D0_N: U39.39 (SDA/AUX-_B)
- new net CSI_CAM_3_D0_P: U39.40 (SCL/AUX+_B)
- new net CSI_CAM_3_D1_N: U39.21 (HPD_B)
- new net CSI_CAM_3_D1_P: U39.20 (CEC_B)
- new net CSI_CAM_4_CLK_N: U40.37 (D0-A)
- new net CSI_CAM_4_CLK_P: U40.38 (D0+A)
- new net CSI_CAM_4_D0_N: U40.35 (D1-A)
- new net CSI_CAM_4_D0_P: U40.36 (D1+A)
- new net CSI_CAM_4_D1_N: U40.33 (D2-A)
- new net CSI_CAM_4_D1_P: U40.34 (D2+A)
- new net CSI_CAM_5_CLK_N: U40.31 (D3-A)
- new net CSI_CAM_5_CLK_P: U40.32 (D3+A)
- new net CSI_CAM_5_D0_N: U40.41 (SDA/AUX-_A)
- new net CSI_CAM_5_D0_P: U40.42 (SCL/AUX+_A)
- new net CSI_CAM_5_D1_N: U40.19 (HPD_A)
- new net CSI_CAM_5_D1_P: U40.18 (CEC_A)
- new net CSI_CAM_6_CLK_N: U40.28 (D0-B)
- new net CSI_CAM_6_CLK_P: U40.29 (D0+B)
- new net CSI_CAM_6_D0_N: U40.26 (D1-B)
- new net CSI_CAM_6_D0_P: U40.27 (D1+B)
- new net CSI_CAM_6_D1_N: U40.24 (D2-B)
- new net CSI_CAM_6_D1_P: U40.25 (D2+B)
- new net CSI_CAM_7_CLK_N: U40.22 (D3-B)
- new net CSI_CAM_7_CLK_P: U40.23 (D3+B)
- new net CSI_CAM_7_D0_N: U40.39 (SDA/AUX-_B)
- new net CSI_CAM_7_D0_P: U40.40 (SCL/AUX+_B)
- new net CSI_CAM_7_D1_N: U40.21 (HPD_B)
- new net CSI_CAM_7_D1_P: U40.20 (CEC_B)
- new net CSI_MUX_EN: R148.2, R149.2, U39.2 (EN), U40.2 (EN)
- no-connect marks 36 -> 0
Other:
- note removed: "AVAILABLE CSI CONFIGURATIONS:"
- note removed: "CONNECTOR J7"
- note removed: "CONNECTOR J8"
- note removed: "CSI Mux"
- note removed: "CSI connector J7"
- note removed: "CSI connector J8"
- note removed: "CSI0 x2"
- note removed: "CSI0 x4"
- note removed: "CSI0x2 CSI2x2"
- note removed: "CSI0x2 CSI2x4"
- note removed: "CSI0x4 CSI2x2"
- note removed: "CSI0x4 CSI2x4"
- note removed: "CSI1 x2"
- note removed: "CSI1x2"
- note removed: "CSI2 x2"
- note removed: "CSI2 x4"
- note removed: "CSI3 x2"
- note removed: "CSI3x2"
- note removed: "CSI3x2 CSI1x2"
- note removed: "NONE"
- note removed: "TO CONNECTOR J7"
- note removed: "TO CONNECTOR J8"
- moved on the sheet: C42, C43, C90, C91, R10, R174, R179, R180, R193, R194, R48, R6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

Commit message: little changes that day
Other:
- moved on the sheet: C131, C132, C133, C135, C42, C43, C88, C90, C91, C92, R10, R105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

Commit message: changement vers gmsl2 en cours
Parts:
- added U35: MAX9296A, symbol GMSL:MAX9296A
Other:
- moved on the sheet: C100, C101, C131, C132, C133, C135, C42, C43, C88, C89, C90, C91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

Commit message: Schematic check
Include Pinmux and Schematic Check excels in doc folder and doing a lot of checking and correcting things.
Parts:
- removed C100, C101, C131, C132, C42, C43, C88, C89, C90, C91, C92, C96, C97: C_100n_0402, jetson-orin-baseboard-footprints:0402-cap, symbol jetson-orin-baseboard:C_100n_0402
- removed C133, C135: 1u, symbol Device:C
- removed R10, R123, R127, R145, R146, R7, R8, R9: R_4k7_0402, jetson-orin-baseboard-footprints:0402-res, symbol jetson-orin-baseboard:R_4k7_0402
- removed R105, R142, R180, R6: R_100k_0402, jetson-orin-baseboard-footprints:0402-res, symbol jetson-orin-baseboard:R_100k_0402
- removed R117, R129, R144, R163, R193, R194, R66, R67, R78: R_10k_0402, jetson-orin-baseboard-footprints:0402-res, symbol jetson-orin-baseboard:R_10k_0402
- removed R148, R149, R50, R51: 10k, symbol Device:R
- removed R161, R162, R166, R167, R168, R171, R174, R179, R47, R49, R74, R76: R_0R_0402, jetson-orin-baseboard-footprints:0402-res, symbol jetson-orin-baseboard:R_0R_0402
- removed R36, R48, R52, R77: 4x2k2_0201_array, jetson-orin-baseboard-footprints:EXB18V, symbol jetson-orin-baseboard:4x2k2_0201_array
- removed U11, U23, U24, U25, U27, U28, U36, U9: AP22615, jetson-orin-baseboard-footprints:TSOT23-6, symbol jetson-orin-baseboard:AP22615
- removed U26: PI4MSD5V9548AZDEX, jetson-orin-baseboard-footprints:VQFN-24, symbol jetson-orin-baseboard:PI4MSD5V9548AZDEX
- removed U31, U32: NTS0102GT, jetson-orin-baseboard-footprints:PSON50P100X195X50-8N, symbol jetson-orin-baseboard:NTS0102GT
- removed U35: MAX9296A, symbol GMSL:MAX9296A
- removed U39, U40: TS3DV642RUARQ1, jetson-orin-baseboard-footprints:WQFN-42-1EP_3.5x9mm_P0.5mm_EP2.05x7.55mm, symbol jetson-orin-baseboard:TS3DV642RUARQ1
- added C84, C85: 0.1u, symbol Device:C
- added D18, D19, D20, D21, D22, D23, D24, D25, D38, D39, D40, D41, D42, D43, D44, D45, D46, D47, D48, D49, D50, D51, D52, D54: Zener, symbol Device:D_Zener
- added J11, J13: F32R-1A7H1-11022, F32R-1A7H1-11022:AMPHENOL_F32R-1A7H1-11022, symbol F32R-1A7H1-11022:F32R-1A7H1-11022
- added R10, R26, R8, R9: 1k, symbol Device:R
- added R36, R40: R_0R_0402, jetson-orin-baseboard-footprints:R_0402_1005Metric, symbol jetson-orin-baseboard:R_0R_0402
- added R6: 10k, symbol Device:R
- added R7: 0, symbol Device:R
- added U11, U3: SN74LV1T125DCKR, SN74LV1T125DCKR:SOT65P210X110-5N, symbol SN74LV1T125DCKR:SN74LV1T125DCKR
- added U9: TS3USB30ERSWR, TS3USB30ERSWR:QFN40P140X180X55-10N, symbol TS3USB30ERSWR:TS3USB30ERSWR
Connections:
- net +3V3: now also C84.1, C85.1, J11.1, J13.1, R10.1, R26.1, R8.1, R9.1, U11.5 (VCC), U3.5 (VCC), U9.9 (VCC)
- net CSI0_CLK_N: now also D22.1 (K), J11.15
- net CSI0_CLK_P: now also D23.1 (K), J11.14
- net CSI0_D0_N: now also D18.1 (K), J11.21
- net CSI0_D0_P: now also D19.1 (K), J11.20
- net CSI0_D1_N: now also D20.1 (K), J11.18
- net CSI0_D1_P: now also D21.1 (K), J11.17
- net CSI1_D0_N: now also D24.1 (K), J11.12
- net CSI1_D0_P: now also D25.1 (K), J11.11
- net CSI1_D1_N: now also D38.1 (K), J11.9
- net CSI1_D1_P: now also D39.1 (K), J11.8
- net CSI2_CLK_N: now also D46.1 (K), J13.15
- net CSI2_CLK_P: now also D47.1 (K), J13.14
- net CSI2_D0_N: now also D42.1 (K), J13.21
- net CSI2_D0_P: now also D43.1 (K), J13.20
- net CSI2_D1_N: now also D44.1 (K), J13.18
- net CSI2_D1_P: now also D45.1 (K), J13.17
- net CSI3_D0_N: now also D48.1 (K), J13.12
- net CSI3_D0_P: now also D49.1 (K), J13.11
- net CSI3_D1_N: now also D50.1 (K), J13.9
- net CSI3_D1_P: now also D51.1 (K), J13.8
- net GND: now also C84.2, C85.2, D18.2 (A), D19.2 (A), D20.2 (A), D21.2 (A), D22.2 (A), D23.2 (A), D24.2 (A), D25.2 (A), D38.2 (A), D39.2 (A), D40.2 (A), D41.2 (A), D42.2 (A), D43.2 (A), D44.2 (A), D45.2 (A), D46.2 (A), D47.2 (A), D48.2 (A), D49.2 (A), D50.2 (A), D51.2 (A), D52.2 (A), D54.2 (A), J11.10, J11.13, J11.16, J11.19, J11.22, J11.4, J11.7, J13.10, J13.13, J13.16, J13.19, J13.22, J13.4, J13.7, R6.1, R7.2, U11.1, U11.3 (GND), U3.1, U3.3 (GND), U9.4 (GND)
- net SCL_CAM: now also R36.2
- net SDA_CAM: now also R40.2
- new net: R40.1, U9.5 (D-)
- new net: R36.1, U9.3 (D+)
- new net: D40.1 (K), J11.6, U3.4
- new net: R7.1, U9.8 (~OE)
- new net: D52.1 (K), J13.6, U11.4
- new net CAM0_I2C_SCL: J11.3, R26.2, U9.1 (D1+)
- new net CAM0_I2C_SDA: J11.2, R9.2, U9.7 (D1-)
- new net CAM0_MCLK: D41.1 (K), J11.5
- new net CAM0_PWDN: U3.2
- new net CAM1_I2C_SCL: J13.3, R8.2, U9.2 (D2+)
- new net CAM1_I2C_SDA: J13.2, R10.2, U9.6 (D2-)
- new net CAM1_MCLK: D54.1 (K), J13.5
- new net CAM1_PWDN: U11.2
- new net CAM_MUX_SEL: R6.2, U9.10 (S)
Other:
- note removed: "ALL SWITCHES 1.5A CURRENT LIMIT"
- note removed: "I2C Mux"
- note removed: "Level shifters"
- note removed: "Power switches"

Commit message: Schematic Done
Other:
- moved on the sheet: R10, R26, R36, R40, R6, R7, R8, R9, U9
