File: jetson-orin-baseboard.kicad_sch (KiCad schematic)
At the start: 4 parts

Commit message: Schematic Done
Other:
- note removed: "Things Left to check: -Check USB-C HPD circuit in SOM page -Check Ethernet DS to confirm layout -Compare USB-C schematics with datasheets and jetson-orin-baseboard pdf -Recheck Peripherals -Check IMU with DS -Check 4G with DS -Understand whole supply schematic"
Changed lines of the file:
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@@
     (effects (font (size 5 5) (thickness 0.4) bold) (justify left bottom))
-  )
-  (text "Things Left to check:\n-Check USB-C HPD circuit in SOM page\n-Check Ethernet DS to confirm layout\n-Compare USB-C schematics with datasheets and jetson-orin-baseboard pdf\n-Recheck Peripherals\n-Check IMU with DS\n-Check 4G with DS\n-Understand whole supply schematic"
-    (at 164.465 41.91 0)
-    (effects (font (size 1.27 1.27)) (justify left bottom))
   )
   (symbol (lib_id "jetson-orin-baseboard:GND") (at 383.54 246.38 0) (unit 1)
