File: jetson-orin-baseboard.kicad_pcb (KiCad board)
At the start: 8 copper layers, 120 x 60 mm, 443 parts, among them J1 533980471, J10 532611071, J11 ERF8-020-05.0-S-DV-L-TR, J12 XT30PW-M, J13 SIM8066-6-1-14-01-A_REVA, J14 SIM7600X-M2-B, J2 1-2199230-6, J3 WE_632723300011_alt_symbol, J4 WE_632723300011_alt_symbol, J5 ARJM11C7-502-AB-ER2-T, J6 F32R-1A7H1-11022, J7 F32R-1A7H1-11022, J8 TC2050-IDC-NL, J9 533980471, M2 M2_2280, Q1 PJE138K, Q10 PJE138K, Q11 PJE138K, Q12 PJE138K, Q13 SSM3J332R, Q2 PJE138K, Q3 PJE138K, Q4 PJE138K, Q5 PJE138K, Q6 BCM857BS-7-F, Q7 PJE138K, Q8 SSM3J332R, Q9 SSM3J332R, SW1 PCM12SMTR, U1 NTS0102GT, U10 TPD4E05U06QDQARQ1, U11 TPD4E05U06QDQARQ1, U12 HD3SS3220, U13 AP22615, U14 TPD4E05U06QDQARQ1, U15 TPD4E05U06QDQARQ1, U16 TPD4E05U06QDQARQ1, U17 TS3USB30ERSWR, U18 SN74LV1T125DCKR, U19 SN74LV1T125DCKR, U2 TPS65987, U20 NTS0102GT, U21 ICM-20602, U22 74LVC2G14GV, U23 74LVC1G175GV, U24 TPS56C230, U25 TPS56C230, U26 NCP730BMT330TBG, U27 TPS7A0518PDBVT, U3 W25Q80DVUXIE_TR, U4 NCP730BMT330TBG, U5 FT230XQ-R, U6 TUSB1046-DCI, U7 TPD4E05U06QDQARQ1, U8 AP22615, U9 TPD4E05U06QDQARQ1, Y1 ECS-327MVATX-2-CN-TR3

Commit message: Copiage de placement composantes part 2
Parts:
- C107, C108, C117, C118, C90, C91, C93, C95, D39, D40, D47, D48, D54, D55, Q10, Q12, Q13, Q7, R120, R124, R125, R126, R128, R132, R133, R148, R151, R152, R153, R154, SW1, TP24, TP25, TP26, U22, U23, U26, U27: moved to B.Cu
- moved R148 218.9 mm to (57.2, 84.0), turned to 90 degrees
- moved U27 213.9 mm to (59.6, 83.8)
- moved C107 211.0 mm to (62.0, 86.9), turned to 90 degrees
- moved Q12 210.5 mm to (59.2, 87.1), turned to -90 degrees
- moved R154 208.3 mm to (60.9, 90.7), turned to 180 degrees
- moved C118 208.0 mm to (62.6, 84.0), turned to 180 degrees
- moved Q13 205.1 mm to (60.2, 93.5), turned to 180 degrees
- moved R153 205.0 mm to (62.9, 82.7)
- moved D55 204.3 mm to (64.0, 85.0)
- moved D52 203.6 mm to (64.2, 85.2), turned to 180 degrees
- moved D54 202.8 mm to (69.8, 81.0), turned to -90 degrees
- moved R149 202.4 mm to (68.6, 86.4), turned to 180 degrees
- moved C115 199.7 mm to (67.8, 99.4), turned to -90 degrees
- moved R151 199.4 mm to (70.9, 79.4), turned to 0 degrees
- moved C108 199.2 mm to (76.3, 79.5), turned to 90 degrees
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
Commit message: copying positions part 4
Parts:
- C100, C28, C33, C35, C45, C50, C51, C53, C60, C61, D11, D4, D5, D6, D7, D8, D9, Q3, R11, R13, R134, R135, R14, R15, R16, R17, R19, R20, R21, R22, R23, R24, R25, R26, R27, R28, R32, R33, R34, R35, R36, R37, R38, R39, R40, R44, R45, R46, R47, R48, R49, R50, R59, R60, R62, R63, R71, R75, R76, R81, R88, R89, R90, R91, TP10, TP11, TP12, TP13, TP14, TP15, TP17, TP20, TP6, TP7, TP8, TP9, U4, U5: moved to B.Cu
- e: renamed from TP18; moved to B.Cu
- moved TP14 176.1 mm to (60.1, 102.4), turned to -45 degrees
- moved TP12 175.1 mm to (59.2, 104.0), turned to -45 degrees
- moved TP13 174.3 mm to (60.0, 103.4), turned to -45 degrees
- moved R20 174.0 mm to (59.8, 97.2)
- moved R55 172.9 mm to (65.0, 113.1), turned to -90 degrees
- moved R19 172.7 mm to (61.1, 98.5), turned to -90 degrees
- moved R56 172.7 mm to (65.5, 116.3), turned to -90 degrees
- moved R57 171.9 mm to (66.5, 119.0), turned to 90 degrees
- moved TP15 171.7 mm to (64.2, 97.2), turned to 180 degrees
- moved D7 171.4 mm to (44.2, 127.0), turned to 0 degrees
- moved R58 170.5 mm to (67.5, 119.0), turned to 90 degrees
- moved R39 170.1 mm to (43.6, 124.2)
- moved R24 167.1 mm to (59.1, 99.2), turned to -90 degrees
- moved R61 166.8 mm to (69.2, 124.8)
- moved TP16 166.8 mm to (71.9, 109.9)
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